File: Driver.sch (KiCad schematic (older format))
At the start: 16 parts, among them U1 TMC2130

Commit message: Initial layout of 1-driver
Changed lines of the file:
@@
 $Descr A4 11693 8268
 encoding utf-8
-Sheet 2 5
+Sheet 4 6
 Title ""
 Date ""
@@
 Connection ~ 4500 5250
 $Comp
-L GND #PWR04
+L GND #PWR09
 U 1 1 59D575B4
 P 4500 5425
-AR Path="/59D57483/59D575B4" Ref="#PWR04"  Part="1"
-AR Path="/59D6DD9D/59D575B4" Ref="#PWR040"  Part="1"
-AR Path="/59D73507/59D575B4" Ref="#PWR031"  Part="1"
-AR Path="/59D73549/59D575B4" Ref="#PWR022"  Part="1"
-F 0 "#PWR04" H 4500 5175 50  0001 C CNN
+AR Path="/59D57483/59D575B4" Ref="#PWR09"  Part="1"
+AR Path="/59D6DD9D/59D575B4" Ref="#PWR027"  Part="1"
+AR Path="/59D73507/59D575B4" Ref="#PWR036"  Part="1"
+AR Path="/59D73549/59D575B4" Ref="#PWR045"  Part="1"
+F 0 "#PWR09" H 4500 5175 50  0001 C CNN
 F 1 "GND" H 4500 5275 50  0000 C CNN
 F 2 "" H 4500 5425 50  0000 C CNN
@@
 	4525 2025 4575 2025
 $Comp
-L GND #PWR05
+L GND #PWR010
 U 1 1 59D588E8
 P 4150 2400
-AR Path="/59D57483/59D588E8" Ref="#PWR05"  Part="1"
-AR Path="/59D6DD9D/59D588E8" Ref="#PWR041"  Part="1"
-AR Path="/59D73507/59D588E8" Ref="#PWR032"  Part="1"
-AR Path="/59D73549/59D588E8" Ref="#PWR023"  Part="1"
-F 0 "#PWR05" H 4150 2150 50  0001 C CNN
+AR Path="/59D57483/59D588E8" Ref="#PWR010"  Part="1"
+AR Path="/59D6DD9D/59D588E8" Ref="#PWR028"  Part="1"
+AR Path="/59D73507/59D588E8" Ref="#PWR037"  Part="1"
+AR Path="/59D73549/59D588E8" Ref="#PWR046"  Part="1"
+F 0 "#PWR010" H 4150 2150 50  0001 C CNN
 F 1 "GND" H 4150 2250 50  0000 C CNN
 F 2 "" H 4150 2400 50  0000 C CNN
@@
 	3125 2875 4575 2875
 $Comp
-L GND #PWR06
+L GND #PWR011
 U 1 1 59D58FC7
 P 4450 3100
-AR Path="/59D57483/59D58FC7" Ref="#PWR06"  Part="1"
-AR Path="/59D6DD9D/59D58FC7" Ref="#PWR042"  Part="1"
-AR Path="/59D73507/59D58FC7" Ref="#PWR033"  Part="1"
-AR Path="/59D73549/59D58FC7" Ref="#PWR024"  Part="1"
-F 0 "#PWR06" H 4450 2850 50  0001 C CNN
+AR Path="/59D57483/59D58FC7" Ref="#PWR011"  Part="1"
+AR Path="/59D6DD9D/59D58FC7" Ref="#PWR029"  Part="1"
+AR Path="/59D73507/59D58FC7" Ref="#PWR038"  Part="1"
+AR Path="/59D73549/59D58FC7" Ref="#PWR047"  Part="1"
+F 0 "#PWR011" H 4450 2850 50  0001 C CNN
 F 1 "GND" H 4450 2950 50  0000 C CNN
 F 2 "" H 4450 3100 50  0000 C CNN
@@
 	4175 2775 4575 2775
 $Comp
-L GND #PWR07
+L GND #PWR012
 U 1 1 59D59F85
 P 4175 3100
-AR Path="/59D57483/59D59F85" Ref="#PWR07"  Part="1"
-AR Path="/59D6DD9D/59D59F85" Ref="#PWR043"  Part="1"
-AR Path="/59D73507/59D59F85" Ref="#PWR034"  Part="1"
-AR Path="/59D73549/59D59F85" Ref="#PWR025"  Part="1"
-F 0 "#PWR07" H 4175 2850 50  0001 C CNN
+AR Path="/59D57483/59D59F85" Ref="#PWR012"  Part="1"
+AR Path="/59D6DD9D/59D59F85" Ref="#PWR030"  Part="1"
+AR Path="/59D73507/59D59F85" Ref="#PWR039"  Part="1"
+AR Path="/59D73549/59D59F85" Ref="#PWR048"  Part="1"
+F 0 "#PWR012" H 4175 2850 50  0001 C CNN
 F 1 "GND" H 4175 2950 50  0000 C CNN
 F 2 "" H 4175 3100 50  0000 C CNN
@@
 $EndComp
 $Comp
-L GND #PWR08
+L GND #PWR013
 U 1 1 59D5A0EE
 P 3925 3100
-AR Path="/59D57483/59D5A0EE" Ref="#PWR08"  Part="1"
-AR Path="/59D6DD9D/59D5A0EE" Ref="#PWR044"  Part="1"
-AR Path="/59D73507/59D5A0EE" Ref="#PWR035"  Part="1"
-AR Path="/59D73549/59D5A0EE" Ref="#PWR026"  Part="1"
-F 0 "#PWR08" H 3925 2850 50  0001 C CNN
+AR Path="/59D57483/59D5A0EE" Ref="#PWR013"  Part="1"
+AR Path="/59D6DD9D/59D5A0EE" Ref="#PWR031"  Part="1"
+AR Path="/59D73507/59D5A0EE" Ref="#PWR040"  Part="1"
+AR Path="/59D73549/59D5A0EE" Ref="#PWR049"  Part="1"
+F 0 "#PWR013" H 3925 2850 50  0001 C CNN
 F 1 "GND" H 3925 2950 50  0000 C CNN
 F 2 "" H 3925 3100 50  0000 C CNN
@@
 $EndComp
 $Comp
-L GND #PWR09
+L GND #PWR014
 U 1 1 59D5A45A
 P 3825 2400
-AR Path="/59D57483/59D5A45A" Ref="#PWR09"  Part="1"
-AR Path="/59D6DD9D/59D5A45A" Ref="#PWR045"  Part="1"
-AR Path="/59D73507/59D5A45A" Ref="#PWR036"  Part="1"
-AR Path="/59D73549/59D5A45A" Ref="#PWR027"  Part="1"
-F 0 "#PWR09" H 3825 2150 50  0001 C CNN
+AR Path="/59D57483/59D5A45A" Ref="#PWR014"  Part="1"
+AR Path="/59D6DD9D/59D5A45A" Ref="#PWR032"  Part="1"
+AR Path="/59D73507/59D5A45A" Ref="#PWR041"  Part="1"
+AR Path="/59D73549/59D5A45A" Ref="#PWR050"  Part="1"
+F 0 "#PWR014" H 3825 2150 50  0001 C CNN
 F 1 "GND" H 3825 2250 50  0000 C CNN
 F 2 "" H 3825 2400 50  0000 C CNN
@@
 $EndComp
 $Comp
-L GND #PWR010
+L GND #PWR015
 U 1 1 59D5A486
 P 3525 2400
-AR Path="/59D57483/59D5A486" Ref="#PWR010"  Part="1"
-AR Path="/59D6DD9D/59D5A486" Ref="#PWR046"  Part="1"
-AR Path="/59D73507/59D5A486" Ref="#PWR037"  Part="1"
-AR Path="/59D73549/59D5A486" Ref="#PWR028"  Part="1"
-F 0 "#PWR010" H 3525 2150 50  0001 C CNN
+AR Path="/59D57483/59D5A486" Ref="#PWR015"  Part="1"
+AR Path="/59D6DD9D/59D5A486" Ref="#PWR033"  Part="1"
+AR Path="/59D73507/59D5A486" Ref="#PWR042"  Part="1"
+AR Path="/59D73549/59D5A486" Ref="#PWR051"  Part="1"
+F 0 "#PWR015" H 3525 2150 50  0001 C CNN
 F 1 "GND" H 3525 2250 50  0000 C CNN
 F 2 "" H 3525 2400 50  0000 C CNN
@@
 $EndComp
 $Comp
-L GND #PWR011
+L GND #PWR016
 U 1 1 59D5A642
 P 3200 2400
-AR Path="/59D57483/59D5A642" Ref="#PWR011"  Part="1"
-AR Path="/59D6DD9D/59D5A642" Ref="#PWR047"  Part="1"
-AR Path="/59D73507/59D5A642" Ref="#PWR038"  Part="1"
-AR Path="/59D73549/59D5A642" Ref="#PWR029"  Part="1"
-F 0 "#PWR011" H 3200 2150 50  0001 C CNN
+AR Path="/59D57483/59D5A642" Ref="#PWR016"  Part="1"
+AR Path="/59D6DD9D/59D5A642" Ref="#PWR034"  Part="1"
+AR Path="/59D73507/59D5A642" Ref="#PWR043"  Part="1"
+AR Path="/59D73549/59D5A642" Ref="#PWR052"  Part="1"
+F 0 "#PWR016" H 3200 2150 50  0001 C CNN
 F 1 "GND" H 3200 2250 50  0000 C CNN
 F 2 "" H 3200 2400 50  0000 C CNN
@@
 	5775 3750 5775 3725
 $Comp
-L GND #PWR012
+L GND #PWR017
 U 1 1 59D5B8C5
 P 6600 3175
-AR Path="/59D57483/59D5B8C5" Ref="#PWR012"  Part="1"
-AR Path="/59D6DD9D/59D5B8C5" Ref="#PWR048"  Part="1"
-AR Path="/59D73507/59D5B8C5" Ref="#PWR039"  Part="1"
-AR Path="/59D73549/59D5B8C5" Ref="#PWR030"  Part="1"
-F 0 "#PWR012" H 6600 2925 50  0001 C CNN
+AR Path="/59D57483/59D5B8C5" Ref="#PWR017"  Part="1"
+AR Path="/59D6DD9D/59D5B8C5" Ref="#PWR035"  Part="1"
+AR Path="/59D73507/59D5B8C5" Ref="#PWR044"  Part="1"
+AR Path="/59D73549/59D5B8C5" Ref="#PWR053"  Part="1"
+F 0 "#PWR017" H 6600 2925 50  0001 C CNN
 F 1 "GND" H 6600 3025 50  0000 C CNN
 F 2 "" H 6600 3175 50  0000 C CNN
@@
 AR Path="/59D73507/59D5D372" Ref="C33"  Part="1"
 AR Path="/59D73549/59D5D372" Ref="C44"  Part="1"
-F 0 "C11" H 6735 3070 50  0000 L CNN
+F 0 "C11" H 6575 3150 50  0000 L CNN
 F 1 "100nF" H 6735 2920 50  0001 L CNN
 F 2 "Capacitors_SMD:C_0603_HandSoldering" H 6725 3000 50  0001 C CNN
